File: pcb/Buttons.kicad_sch (KiCad schematic)
At the start: 3 parts, among them SW1 POWER/MODE, SW2 LEFT, SW3 RIGHT

Commit message: Finished First Version
Parts:
- SW1: value POWER/MODE -> KMR211
- SW2: value LEFT -> KMR211
- SW3: value RIGHT -> KMR211
Changed lines of the file:
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@@
       (effects (font (size 1.27 1.27)) (justify right))
     )
-    (property "Value" "POWER/MODE" (id 1) (at 87.63 66.0399 90)
+    (property "Value" "KMR211" (id 1) (at 87.63 66.0399 90)
       (effects (font (size 1.27 1.27)) (justify right))
     )
@@
       (effects (font (size 1.27 1.27)) (justify right))
     )
-    (property "Value" "RIGHT" (id 1) (at 120.65 66.0399 90)
+    (property "Value" "KMR211" (id 1) (at 120.65 66.0399 90)
       (effects (font (size 1.27 1.27)) (justify right))
     )
@@
       (effects (font (size 1.27 1.27)) (justify right))
     )
-    (property "Value" "LEFT" (id 1) (at 105.41 66.0399 90)
+    (property "Value" "KMR211" (id 1) (at 105.41 66.0399 90)
       (effects (font (size 1.27 1.27)) (justify right))
     )
