File: pcb/LEDs.kicad_sch (KiCad schematic)
At the start: 0 parts

Commit message: Finished First Version
Parts:
- added C16, C17, C18, C19, C20, C21: 4.7uF, Capacitor_SMD:C_0603_1608Metric, symbol Device:C
Connections:
- net GND: now also C16.2, C17.2, C18.2, C19.2, C20.2, C21.2
- net V_{DD}: now also C16.1, C17.1, C18.1, C19.1, C20.1, C21.1
