File: pcb/MCU.kicad_sch (KiCad schematic)
At the start: 20 parts, among them SW4 RESET, U3 ESP32-C3, U4 SN74LVC1T45DBV, Y1 32.768kHz 12.5pF, Y2 40MHz 12pF

Commit message: Finished First Version
Parts:
- SW4: value RESET -> EVQ-PUM02K
Changed lines of the file:
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@@
       (effects (font (size 1.27 1.27)) (justify right))
     )
-    (property "Value" "RESET" (id 1) (at 62.23 86.3599 90)
+    (property "Value" "EVQ-PUM02K" (id 1) (at 62.23 86.3599 90)
       (effects (font (size 1.27 1.27)) (justify right))
     )
